File: EAGLE/Project/Project_Amp_RevA.sch (EAGLE design)
At the start: 66 parts, among them J1 Guitar Input, J2 CD Input, J3 Line Out, U1 OPA2314, U2 OPA2314, U3 OPA2314, U4 OPA2314, U5 TS3A5018, U6 OPA2314, U7 OPA2314

Commit message: Include EAGLE project files
Other:
- moved on the sheet: BT1, BT2, C1, C10, C11, C12, C13, C14, C2, C3, C4, C5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
